File: hardware/P3DA.brd (EAGLE design)
At the start: 78.7 x 66 mm, 70 parts, among them J2 22-27-2041-04, J3 22-27-2041-04, J4 22-27-2041-04, J5 22-27-2041-04, J6 22-27-2041-04, J7 22-27-2041-04, X7 9090-4R

Commit message: Refactoring PCB and schematic
Parts:
- removed U$1: TSOP1738, tsop:TSOP17XX
- added IR1: TSOP1756TB1, telefunken:TSOP17_TB1
- ARDUINO: value ARDUINO_NANO2 -> NANO
- C1, C3: value (none) -> 0.1
- C2: value (none) -> 100u
- moved R38 2.62 mm to (29.2, 62.2)
- moved R37 1.80 mm to (26.0, 64.8)
- turned R1 to 180 degrees
- turned R11 to 180 degrees
- turned R13 to 180 degrees
- turned R15 to 180 degrees
- turned R17 to 180 degrees
- turned R19 to 0 degrees
- turned R21 to 0 degrees
- turned R23 to 0 degrees
- turned R25 to 0 degrees
- turned R27 to 0 degrees
- turned R29 to 0 degrees
- turned R3 to 180 degrees
- turned R31 to 0 degrees
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- renumbered MODUL1 to ARDUINO
Connections:
- removed net B1_PWM: ARDUINO.J1.5, R5.1
- removed net B2_PWM: ARDUINO.J1.8, R11.1
- removed net B3_PWM: ARDUINO.J1.11, R17.1
- removed net B4_PWM: ARDUINO.J2.9, R23.1
- removed net B5_PWM: ARDUINO.J2.12, R29.1
- removed net B6_PWM: ARDUINO.J1.15, R35.1
- removed net G1_PWM: ARDUINO.J1.7, R3.1
- removed net G2_PWM: ARDUINO.J1.10, R9.1
- removed net G3_PWM: ARDUINO.J1.13, R15.1
- removed net G4_PWM: ARDUINO.J2.7, R21.1
- removed net G5_PWM: ARDUINO.J2.10, R27.1
- removed net G6_PWM: ARDUINO.J2.15, R33.1
- removed net N$1: R1.2, R2.2, T1.3
- removed net N$4: R3.2, R4.2, T2.3
- removed net R1_PWM: ARDUINO.J1.6, R1.1
- removed net R2_PWM: ARDUINO.J1.9, R7.1
- removed net R3_PWM: ARDUINO.J1.12, R13.1
- removed net R4_PWM: ARDUINO.J2.8, R19.1
- removed net R5_PWM: ARDUINO.J2.11, R25.1
- removed net R6_PWM: ARDUINO.J1.14, R31.1
- new net B_IN1: ARDUINO.J1.5, R5.2
- new net B_IN2: ARDUINO.J1.8, R11.2
- new net B_IN3: ARDUINO.J1.11, R17.2
- new net B_IN4: ARDUINO.J2.9, R23.2
- new net B_IN5: ARDUINO.J2.12, R29.2
- new net B_IN6: ARDUINO.J1.15, R35.2
- new net G_IN1: ARDUINO.J1.7, R3.2
- new net G_IN2: ARDUINO.J1.10, R9.2
- new net G_IN3: ARDUINO.J1.13, R15.2
- new net G_IN4: ARDUINO.J2.7, R21.2
- new net G_IN5: ARDUINO.J2.10, R27.2
- new net G_IN6: ARDUINO.J2.15, R33.2
- new net N$19: R1.1, R2.2, T1.3
- new net N$20: R3.1, R4.2, T2.3
- new net R_IN1: ARDUINO.J1.6, R1.2
- new net R_IN2: ARDUINO.J1.9, R7.2
- new net R_IN3: ARDUINO.J1.12, R13.2
- new net R_IN4: ARDUINO.J2.8, R19.2
- new net R_IN5: ARDUINO.J2.11, R25.2
- new net R_IN6: ARDUINO.J1.14, R31.2
- net +5V: now also IR1.VS; no longer U$1.V+
- net GND: now also IR1.GND, J1.1; no longer U$1.GND
- net IR: now also IR1.VO; no longer U$1.OUT
- net N$10: now also R19.1; no longer R19.2
- net N$11: now also R21.1; no longer R21.2
- net N$12: now also R23.1; no longer R23.2
- net N$13: now also R25.1; no longer R25.2
- net N$14: now also R27.1; no longer R27.2
- net N$15: now also R29.1; no longer R29.2
- net N$16: now also R31.1; no longer R31.2
- net N$17: now also R33.1; no longer R33.2
- net N$18: now also R35.1; no longer R35.2
- net N$2: now also R7.1; no longer R7.2
- net N$3: now also R9.1; no longer R9.2
- net N$5: now also R5.1; no longer R5.2
- net N$6: now also R11.1; no longer R11.2
- net N$7: now also R13.1; no longer R13.2
- net N$8: now also R15.1; no longer R15.2
- net N$9: now also R17.1; no longer R17.2
Routing:
- net R_IN6: track 0.00 -> 20.2 mm
- net R6_PWM: track 20.2 -> 0.00 mm
- net B_IN6: track 0.00 -> 20.2 mm
- net B6_PWM: track 20.2 -> 0.00 mm
- net N$20: track 0.00 -> 17.9 mm
- net N$4: track 17.8 -> 0.00 mm
- net N$19: track 0.00 -> 16.8 mm
- net N$1: track 16.8 -> 0.00 mm
- net GND: track 461.3 -> 468.5 mm
- net R_IN5: track 0.00 -> 3.17 mm
- net +5V: track 33.4 -> 30.4 mm
- net R_IN4: track 0.00 -> 2.86 mm
- net R_IN3: track 0.00 -> 2.86 mm
- net R_IN2: track 0.00 -> 2.86 mm
- net R_IN1: track 0.00 -> 2.86 mm
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
Commit message: Add border
Routing:
- net N$1: track 0.00 -> 289.6 mm
Changed lines of the file:
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@@
 <grid distance="0.05" unitdist="inch" unit="inch" style="dots" multiple="1" display="yes" altdistance="0.025" altunitdist="inch" altunit="inch"/>
 <layers>
-<layer number="1" name="Top" color="4" fill="1" visible="yes" active="yes"/>
+<layer number="1" name="Top" color="4" fill="1" visible="no" active="yes"/>
 <layer number="16" name="Bottom" color="1" fill="1" visible="yes" active="yes"/>
 <layer number="17" name="Pads" color="2" fill="1" visible="yes" active="yes"/>
 <layer number="18" name="Vias" color="2" fill="1" visible="yes" active="yes"/>
-<layer number="19" name="Unrouted" color="6" fill="1" visible="yes" active="yes"/>
-<layer number="20" name="Dimension" color="15" fill="1" visible="yes" active="yes"/>
-<layer number="21" name="tPlace" color="7" fill="1" visible="yes" active="yes"/>
-<layer number="22" name="bPlace" color="7" fill="1" visible="yes" active="yes"/>
-<layer number="23" name="tOrigins" color="15" fill="1" visible="yes" active="yes"/>
-<layer number="24" name="bOrigins" color="15" fill="1" visible="yes" active="yes"/>
+<layer number="19" name="Unrouted" color="6" fill="1" visible="no" active="yes"/>
+<layer number="20" name="Dimension" color="15" fill="1" visible="no" active="yes"/>
+<layer number="21" name="tPlace" color="7" fill="1" visible="no" active="yes"/>
+<layer number="22" name="bPlace" color="7" fill="1" visible="no" active="yes"/>
+<layer number="23" name="tOrigins" color="15" fill="1" visible="no" active="yes"/>
+<layer number="24" name="bOrigins" color="15" fill="1" visible="no" active="yes"/>
 <layer number="25" name="tNames" color="7" fill="1" visible="no" active="yes"/>
 <layer number="26" name="bNames" color="7" fill="1" visible="no" active="yes"/>
@@
 <layer number="50" name="dxf" color="7" fill="1" visible="no" active="yes"/>
 <layer number="51" name="tDocu" color="7" fill="1" visible="no" active="yes"/>
-<layer number="52" name="bDocu" color="7" fill="1" visible="yes" active="yes"/>
+<layer number="52" name="bDocu" color="7" fill="1" visible="no" active="yes"/>
 <layer number="56" name="wert" color="7" fill="1" visible="no" active="yes"/>
 <layer number="91" name="Nets" color="2" fill="1" visible="no" active="no"/>
@@
 <wire x1="52.07" y1="36.83" x2="51.755" y2="36.83" width="0.4064" layer="16"/>
 </signal>
+<signal name="N$1">
+<wire x1="0" y1="0" x2="0" y2="66.04" width="0" layer="16"/>
+<wire x1="0" y1="66.04" x2="78.74" y2="66.04" width="0" layer="16"/>
+<wire x1="78.74" y1="66.04" x2="78.74" y2="0" width="0" layer="16"/>
+<wire x1="78.74" y1="0" x2="0" y2="0" width="0" layer="16"/>
+</signal>
 </signals>
